File: hardware/placa_fabricar/Joystick_brd_v1.sch (KiCad schematic (older format))
At the start: 19 parts, among them U1 ProMicro, U2 74LS166, U3 74LS166, U4 74LS166, U5 74LS166, U6 74LS166, U7 74LS166

Commit message: comienzo la pcb, sch casi acabado
Parts:
- added J1, J2, J3, J4, J5, J6, J?: Screw_Terminal_1x08, Pin_Headers:Pin_Header_Straight_1x08_Pitch2.54mm, symbol Screw_Terminal_1x08
- added J10, J11, J12, J7, J8, J9: CONN_02X08, Pin_Headers:Pin_Header_Straight_2x08_Pitch2.54mm, symbol CONN_02X08
- RN1, RN10, RN11, RN12, RN2, RN3, RN4, RN5, RN6, RN7, RN8, RN9: footprint (none) -> Resistors_SMD:R_Array_Convex_4x1206
- U1: footprint (none) -> Teensy:promicro; symbol ProMicro -> ProMicro-RESCUE-Joystick_brd_v1
- U2, U3, U4, U5, U6, U7: footprint (none) -> Housings_SOIC:SOIC-16_3.9x9.9mm_Pitch1.27mm
Connections:
- net GND: now also J10.1 (P1), J10.11 (P11), J10.13 (P13), J10.15 (P15), J10.3 (P3), J10.5 (P5), J10.7 (P7), J10.9 (P9), J11.1 (P1), J11.11 (P11), J11.13 (P13), J11.15 (P15), J11.3 (P3), J11.5 (P5), J11.7 (P7), J11.9 (P9), J12.1 (P1), J12.11 (P11), J12.13 (P13), J12.15 (P15), J12.3 (P3), J12.5 (P5), J12.7 (P7), J12.9 (P9), J7.1 (P1), J7.11 (P11), J7.13 (P13), J7.15 (P15), J7.3 (P3), J7.5 (P5), J7.7 (P7), J7.9 (P9), J8.1 (P1), J8.11 (P11), J8.13 (P13), J8.15 (P15), J8.3 (P3), J8.5 (P5), J8.7 (P7), J8.9 (P9), J9.1 (P1), J9.11 (P11), J9.13 (P13), J9.15 (P15), J9.3 (P3), J9.5 (P5), J9.7 (P7), J9.9 (P9), J?.1, J?.2, J?.3, J?.4, J?.5, J?.6, J?.7, J?.8
- net P4_B4: now reaches RN1.5 (R4.2), U2.5 (D)
- net P4_B4: now also J10.8 (P8), J4.4
- net P4_B3: now reaches RN1.6 (R3.2), U2.4 (C)
- net P4_B3: now also J10.6 (P6), J4.3
- net P4_B2: now reaches RN1.7 (R2.2), U2.3 (B)
- net P4_B2: now also J10.4 (P4), J4.2
- net P4_B1: now reaches RN1.8 (R1.2), U2.2 (A)
- net P4_B1: now also J10.2 (P2), J4.1
- net P4_START: now reaches RN2.5 (R4.2), U2.14 (H)
- net P4_START: now also J10.16 (P16), J4.8
- net P4_COIN: now reaches RN2.6 (R3.2), U2.12 (G)
- net P4_COIN: now also J10.14 (P14), J4.7
- net P4_B6: now reaches RN2.7 (R2.2), U2.11 (F)
- net P4_B6: now also J10.12 (P12), J4.6
- net P4_B5: now reaches RN2.8 (R1.2), U2.10 (E)
- net P4_B5: now also J10.10 (P10), J4.5
- net P3_START: now reaches RN3.5 (R4.2), U3.5 (D)
- net P3_START: now also J11.8 (P8), J5.4
- net P3_COIN: now reaches RN3.6 (R3.2), U3.4 (C)
- net P3_COIN: now also J11.6 (P6), J5.3
- net P3_B6: now reaches RN3.7 (R2.2), U3.3 (B)
- net P3_B6: now also J11.4 (P4), J5.2
- net P3_B5: now reaches RN3.8 (R1.2), U3.2 (A)
- net P3_B5: now also J11.2 (P2), J5.1
- net P4_RG: now reaches RN4.5 (R4.2), U3.14 (H)
- net P4_RG: now also J11.16 (P16), J5.8
- net P4_LF: now reaches RN4.6 (R3.2), U3.12 (G)
- net P4_LF: now also J11.14 (P14), J5.7
- net P4_DW: now reaches RN4.7 (R2.2), U3.11 (F)
- net P4_DW: now also J11.12 (P12), J5.6
- net P4_UP: now reaches RN4.8 (R1.2), U3.10 (E)
- net P4_UP: now also J11.10 (P10), J5.5
- net P2_B4: now reaches RN7.5 (R4.2), U5.5 (D)
- net P2_B4: now also J1.4, J7.8 (P8)
- net P2_B3: now reaches RN7.6 (R3.2), U5.4 (C)
- net P2_B3: now also J1.3, J7.6 (P6)
- net P2_B2: now reaches RN7.7 (R2.2), U5.3 (B)
- net P2_B2: now also J1.2, J7.4 (P4)
- net P2_B1: now reaches RN7.8 (R1.2), U5.2 (A)
- net P2_B1: now also J1.1, J7.2 (P2)
- net P2_START: now reaches RN8.5 (R4.2), U5.14 (H)
- net P2_START: now also J1.8, J7.16 (P16)
- net P2_COIN: now reaches RN8.6 (R3.2), U5.12 (G)
- net P2_COIN: now also J1.7, J7.14 (P14)
- net P2_B6: now reaches RN8.7 (R2.2), U5.11 (F)
- net P2_B6: now also J1.6, J7.12 (P12)
- net P2_B5: now reaches RN8.8 (R1.2), U5.10 (E)
- net P2_B5: now also J1.5, J7.10 (P10)
- net P1_START: now reaches RN9.5 (R4.2), U6.5 (D)
- net P1_START: now also J2.4, J8.8 (P8)
- net P1_COIN: now reaches RN9.6 (R3.2), U6.4 (C)
- net P1_COIN: now also J2.3, J8.6 (P6)
- net P1_B6: now reaches RN9.7 (R2.2), U6.3 (B)
- net P1_B6: now also J2.2, J8.4 (P4)
- net P1_B5: now reaches RN9.8 (R1.2), U6.2 (A)
- net P1_B5: now also J2.1, J8.2 (P2)
- net P2_RG: now reaches RN10.5 (R4.2), U6.14 (H)
- net P2_RG: now also J2.8, J8.16 (P16)
- net P2_LF: now reaches RN10.6 (R3.2), U6.12 (G)
- net P2_LF: now also J2.7, J8.14 (P14)
- net P2_DW: now reaches RN10.7 (R2.2), U6.11 (F)
- net P2_DW: now also J2.6, J8.12 (P12)
- net P2_UP: now reaches RN10.8 (R1.2), U6.10 (E)
- net P2_UP: now also J2.5, J8.10 (P10)
- net P3_RG: now reaches RN5.5 (R4.2), U4.5 (D)
- net P3_RG: now also J12.8 (P8), J6.4
- net P3_LF: now reaches RN5.6 (R3.2), U4.4 (C)
- net P3_LF: now also J12.6 (P6), J6.3
- net P3_DW: now reaches RN5.7 (R2.2), U4.3 (B)
- net P3_DW: now also J12.4 (P4), J6.2
- net P3_UP: now reaches RN5.8 (R1.2), U4.2 (A)
- net P3_UP: now also J12.2 (P2), J6.1
- net P3_B4: now reaches RN6.5 (R4.2), U4.14 (H)
- net P3_B4: now also J12.16 (P16), J6.8
- net P3_B3: now reaches RN6.6 (R3.2), U4.12 (G)
- net P3_B3: now also J12.14 (P14), J6.7
- net P3_B2: now reaches RN6.7 (R2.2), U4.11 (F)
- net P3_B2: now also J12.12 (P12), J6.6
- net P3_B1: now reaches RN6.8 (R1.2), U4.10 (E)
- net P3_B1: now also J12.10 (P10), J6.5
- net P1_RG: now reaches RN11.5 (R4.2), U7.5 (D)
- net P1_RG: now also J3.4, J9.8 (P8)
- net P1_LF: now reaches RN11.6 (R3.2), U7.4 (C)
- net P1_LF: now also J3.3, J9.6 (P6)
- net P1_DW: now reaches RN11.7 (R2.2), U7.3 (B)
- net P1_DW: now also J3.2, J9.4 (P4)
- net P1_UP: now reaches RN11.8 (R1.2), U7.2 (A)
- net P1_UP: now also J3.1, J9.2 (P2)
- net P1_B4: now reaches RN12.5 (R4.2), U7.14 (H)
- net P1_B4: now also J3.8, J9.16 (P16)
- net P1_B3: now reaches RN12.6 (R3.2), U7.12 (G)
- net P1_B3: now also J3.7, J9.14 (P14)
- net P1_B2: now reaches RN12.7 (R2.2), U7.11 (F)
- net P1_B2: now also J3.6, J9.12 (P12)
- net P1_B1: now reaches RN12.8 (R1.2), U7.10 (E)
- net P1_B1: now also J3.5, J9.10 (P10)
Other:
- note added: "JST terminals"
- moved on the sheet: RN1, RN10, RN11, RN12, RN2, RN3, RN4, RN5, RN6, RN7, RN8, RN9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
